Commit message: update l4w4

File: l4w4_description/urdf/l4w4_description.urdf (robot description, URDF)
Before this commit: robot l4w4, 19 links, 18 joints
Links:
- link FL_calf: mass 0.829 -> 1.943; geometry collision box size=0.04 0.03 0.23; collision cylinder length=0.035 radius=0.0405
- link FL_foot: mass 2.6 -> 0.91041; geometry collision mesh filename=package://l4w4_description/meshes/wheel.STL scale=1 1 1; visual mesh filename=package://l4w4_description/meshes/wheel.STL scale=1 1 1
- link FL_hip: mass 2 -> 1.922; geometry collision cylinder length=0.001 radius=0.001; visual mesh filename=package://l4w4_description/meshes/shoulder_left.STL scale=1 1 1
- link FL_thigh: mass 3.396 -> 3.793; geometry collision box size=0.1 0.044 0.3; visual mesh filename=package://l4w4_description/meshes/thigh_left.STL scale=1 1 1
- link FR_calf: mass 0.829 -> 1.943; geometry collision box size=0.04 0.03 0.23; collision cylinder length=0.035 radius=0.0405
- link FR_foot: mass 2.6 -> 0.91041; geometry collision mesh filename=package://l4w4_description/meshes/wheel.STL scale=1 1 1; visual mesh filename=package://l4w4_description/meshes/wheel.STL scale=1 1 1
- link FR_hip: mass 2 -> 1.922; geometry collision cylinder length=0.001 radius=0.001; visual mesh filename=package://l4w4_description/meshes/shoulder_right.STL
- link FR_thigh: mass 3.396 -> 3.793; geometry collision box size=0.1 0.044 0.3; visual mesh filename=package://l4w4_description/meshes/thigh_right.STL scale=1 1 1
- link RL_calf: mass 0.829 -> 1.943; geometry collision box size=0.04 0.03 0.23; collision cylinder length=0.035 radius=0.0405
- link RL_foot: mass 2.6 -> 0.91041; geometry collision mesh filename=package://l4w4_description/meshes/wheel.STL scale=1 1 1; visual mesh filename=package://l4w4_description/meshes/wheel.STL scale=1 1 1
- link RL_hip: mass 2 -> 1.922; geometry collision cylinder length=0.001 radius=0.001; visual mesh filename=package://l4w4_description/meshes/shoulder_left.STL scale=1 1 1
- link RL_thigh: mass 3.396 -> 3.793; geometry collision box size=0.1 0.044 0.3; visual mesh filename=package://l4w4_description/meshes/thigh_left.STL scale=1 1 1
- link RR_calf: mass 0.829 -> 1.943; geometry collision box size=0.04 0.03 0.23; collision cylinder length=0.035 radius=0.0405
- link RR_foot: mass 2.6 -> 0.91041; geometry collision mesh filename=package://l4w4_description/meshes/wheel.STL scale=1 1 1; visual mesh filename=package://l4w4_description/meshes/wheel.STL scale=1 1 1
- link RR_hip: mass 2 -> 1.922; geometry collision cylinder length=0.001 radius=0.001; visual mesh filename=package://l4w4_description/meshes/shoulder_right.STL scale=1 1 1
- link RR_thigh: mass 3.396 -> 3.793; geometry collision box size=0.1 0.044 0.3; visual mesh filename=package://l4w4_description/meshes/thigh_right.STL scale=1 1 1
- link trunk: mass 18.057 -> 18.826; geometry collision box size=0.33 0.016 0.042; collision box size=0.33 0.016 0.042
Joints:
- joint FL_calf_joint: limit lower=-2.7 upper=-0.17 effort=135 velocity=12.56 -> lower=-2.75 upper=-0.9 effort=200 velocity=8.3; origin xyz=0 0.1145 -0.3 rpy=0 0 0 -> xyz=0 0.108 -0.3 rpy=0 0 0
- joint FL_foot_joint: limit lower=-1000000 upper=1000000 effort=32 velocity=12.0 -> lower=-99999 upper=99999 effort=25 velocity=21.0
- joint FL_hip_joint: limit lower=-0.5236 upper=0.5236 effort=110 velocity=11.5 -> lower=-0.5236 upper=0.5236 effort=110 velocity=12.56; origin xyz=0.249 0.065 0 rpy=0 0 0 -> xyz=0.2515 0.07 0 rpy=0 0 0
- joint FL_thigh_joint: limit lower=-1.4 upper=3.14 effort=110 velocity=12.56 -> lower=-1.22 upper=3.8397 effort=110 velocity=12.56
- joint FR_calf_joint: limit lower=-2.7 upper=-0.17 effort=135 velocity=12.56 -> lower=-2.75 upper=-0.9 effort=200 velocity=8.3; origin xyz=0 -0.1145 -0.3 rpy=0 0 0 -> xyz=0 -0.108 -0.3 rpy=0 0 0
- joint FR_foot_joint: limit lower=-1000000 upper=1000000 effort=32 velocity=12.0 -> lower=-99999 upper=99999 effort=25 velocity=21.0
- joint FR_hip_joint: limit lower=-0.5236 upper=0.5236 effort=110 velocity=11.5 -> lower=-0.5236 upper=0.5236 effort=110 velocity=12.56; origin xyz=0.249 -0.065 0 rpy=0 0 0 -> xyz=0.2515 -0.07 0 rpy=0 0 0
- joint FR_thigh_joint: limit lower=-1.4 upper=3.14 effort=110 velocity=12.56 -> lower=-1.22 upper=3.8397 effort=110 velocity=12.56
- joint RL_calf_joint: limit lower=-2.7 upper=-0.17 effort=135 velocity=12.56 -> lower=-2.75 upper=-0.9 effort=200 velocity=8.3; origin xyz=0 0.1145 -0.3 rpy=0 0 0 -> xyz=0 0.108 -0.3 rpy=0 0 0
- joint RL_foot_joint: limit lower=-1000000 upper=1000000 effort=32 velocity=12.0 -> lower=-99999 upper=99999 effort=25 velocity=21.0
- joint RL_hip_joint: limit lower=-0.5236 upper=0.5236 effort=110 velocity=11.5 -> lower=-0.5236 upper=0.5236 effort=110 velocity=12.56; origin xyz=-0.249 0.065 0 rpy=0 0 0 -> xyz=-0.2515 0.07 0 rpy=0 0 0
- joint RL_thigh_joint: limit lower=-1.4 upper=3.14 effort=110 velocity=12.56 -> lower=-1.22 upper=3.8397 effort=110 velocity=12.56
- joint RR_calf_joint: limit lower=-2.7 upper=-0.17 effort=135 velocity=12.56 -> lower=-2.75 upper=-0.9 effort=200 velocity=8.3; origin xyz=0 -0.1145 -0.3 rpy=0 0 0 -> xyz=0 -0.108 -0.3 rpy=0 0 0
- joint RR_foot_joint: limit lower=-1000000 upper=1000000 effort=32 velocity=12.0 -> lower=-99999 upper=99999 effort=25 velocity=21
- joint RR_hip_joint: limit lower=-0.5236 upper=0.5236 effort=110 velocity=11.5 -> lower=-0.5236 upper=0.5236 effort=110 velocity=12.56; origin xyz=-0.249 -0.065 0 rpy=0 0 0 -> xyz=-0.2515 -0.07 0 rpy=0 0 0
- joint RR_thigh_joint: limit lower=-1.4 upper=3.14 effort=110 velocity=12.56 -> lower=-1.22 upper=3.8397 effort=110 velocity=12.56
- joint imu_joint: parent trunk -> base
